File: Schematic/master-gpio.sch (EAGLE design)
At the start: 15 parts, among them T1 BC337, T2 BC337, T3 BC337, T4 BC337

Commit message: GPIO changes
Parts:
- removed R3: 1200, eagle-ltspice:R
- removed R8: 120, eagle-ltspice:R
- added D1: Blue, eagle-ltspice:DIODE_E-
- R1: value 2200 -> 220
Connections:
- net GND: now also D1.A, T3.E; no longer R1.1, R8.1
- net N$3: no longer R8.2
- net N$5: now also R1.1; no longer R3.2
- net VCC: now also D1.C; no longer R3.1
Other:
- moved on the sheet: R1
Changed lines of the file:
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@@
 <part name="SUPPLY3" library="supply2" deviceset="GND" device=""/>
 <part name="SUPPLY4" library="supply2" deviceset="VCC" device=""/>
-<part name="SUPPLY7" library="supply2" deviceset="GND" device=""/>
 <part name="SUPPLY2" library="supply2" deviceset="GND" device=""/>
 <part name="SUPPLY5" library="supply2" deviceset="VCC" device="" value="5V"/>
 <part name="SUPPLY6" library="supply2" deviceset="VCC" device="" value="5V"/>
-<part name="SUPPLY9" library="supply2" deviceset="VCC" device="" value="RX"/>
 <part name="PIN13" library="supply2" deviceset="VCC" device="" value="Pin"/>
 <part name="SUPPLY11" library="supply2" deviceset="VCC" device="" value="TX"/>
-<part name="R1" library="eagle-ltspice" deviceset="R" device="" value="2200"/>
-<part name="R3" library="eagle-ltspice" deviceset="R" device="" value="1200"/>
-<part name="SUPPLY10" library="supply2" deviceset="GND" device=""/>
-<part name="R8" library="eagle-ltspice" deviceset="R" device="" value="120"/>
 <part name="R2" library="eagle-ltspice" deviceset="R" device="" value="120"/>
 <part name="T1" library="transistor" deviceset="BC337" device=""/>
@@
 <part name="R7" library="eagle-ltspice" deviceset="R" device="" value="1000"/>
 <part name="R10" library="eagle-ltspice" deviceset="R" device="" value="1000"/>
+<part name="SUPPLY16" library="supply2" deviceset="GND" device=""/>
+<part name="R1" library="eagle-ltspice" deviceset="R" device="" value="220"/>
+<part name="PIN1" library="supply2" deviceset="VCC" device="" value="Pin"/>
+<part name="SUPPLY7" library="supply2" deviceset="GND" device=""/>
+<part name="D1" library="eagle-ltspice" deviceset="DIODE_E-" device="" value="Blue"/>
 </parts>
 <sheets>
@@
 <instance part="SUPPLY3" gate="GND" x="10.16" y="116.84"/>
 <instance part="SUPPLY4" gate="G$1" x="10.16" y="147.32"/>
-<instance part="SUPPLY7" gate="GND" x="-35.56" y="106.68"/>
 <instance part="SUPPLY2" gate="GND" x="-53.34" y="132.08"/>
 <instance part="SUPPLY5" gate="G$1" x="-63.5" y="127"/>
 <instance part="SUPPLY6" gate="G$1" x="-53.34" y="160.02"/>
-<instance part="SUPPLY9" gate="G$1" x="-40.64" y="152.4" rot="R90"/>
 <instance part="PIN13" gate="G$1" x="-86.36" y="134.62" rot="R90"/>
 <instance part="SUPPLY11" gate="G$1" x="-81.28" y="109.22" rot="R90"/>
-<instance part="R1" gate="G$1" x="-33.02" y="147.32" rot="R90"/>
-<instance part="R3" gate="G$1" x="-33.02" y="157.48" rot="R90"/>
-<instance part="SUPPLY10" gate="GND" x="-33.02" y="139.7"/>
-<instance part="R8" gate="G$1" x="-35.56" y="114.3" rot="R90"/>
 <instance part="R2" gate="G$1" x="2.54" y="132.08" rot="R90"/>
 <instance part="T1" gate="G$1" x="-55.88" y="139.7"/>
@@
 <instance part="R7" gate="G$1" x="-73.66" y="109.22" rot="R180"/>
 <instance part="R10" gate="G$1" x="-78.74" y="134.62" rot="R180"/>
+<instance part="SUPPLY16" gate="GND" x="-63.5" y="101.6"/>
+<instance part="R1" gate="G$1" x="-30.48" y="149.86" rot="R90"/>
+<instance part="PIN1" gate="G$1" x="-43.18" y="154.94" rot="R90"/>
+<instance part="SUPPLY7" gate="GND" x="-38.1" y="142.24"/>
+<instance part="D1" gate="G$1" x="-38.1" y="147.32"/>
 </instances>
 <busses>
@@
 <net name="GND" class="0">
 <segment>
-<pinref part="R1" gate="G$1" pin="1"/>
-<pinref part="SUPPLY10" gate="GND" pin="GND"/>
-</segment>
-<segment>
-<pinref part="R8" gate="G$1" pin="1"/>
-<pinref part="SUPPLY7" gate="GND" pin="GND"/>
-</segment>
-<segment>
 <pinref part="T1" gate="G$1" pin="E"/>
 <pinref part="SUPPLY2" gate="GND" pin="GND"/>
@@
 <pinref part="SUPPLY13" gate="GND" pin="GND"/>
 </segment>
+<segment>
+<pinref part="T3" gate="G$1" pin="E"/>
+<pinref part="SUPPLY16" gate="GND" pin="GND"/>
+</segment>
+<segment>
+<pinref part="SUPPLY7" gate="GND" pin="GND"/>
+<pinref part="D1" gate="G$1" pin="A"/>
+</segment>
 </net>
 <net name="VCC" class="0">
@@
 <segment>
 <pinref part="R1" gate="G$1" pin="2"/>
-<pinref part="R3" gate="G$1" pin="1"/>
-<wire x1="-33.02" y1="152.4" x2="-38.1" y2="152.4" width="0.1524" layer="91"/>
-<pinref part="SUPPLY9" gate="G$1" pin="VCC"/>
-</segment>
-</net>
-<net name="N$5" class="0">
-<segment>
-<pinref part="MASTER" gate="G$1" pin="RO"/>
-<wire x1="-25.4" y1="144.78" x2="-25.4" y2="165.1" width="0.1524" layer="91"/>
-<pinref part="R3" gate="G$1" pin="2"/>
-<wire x1="-25.4" y1="165.1" x2="-33.02" y2="165.1" width="0.1524" layer="91"/>
-<wire x1="-33.02" y1="165.1" x2="-33.02" y2="162.56" width="0.1524" layer="91"/>
+<pinref part="PIN1" gate="G$1" pin="VCC"/>
+<wire x1="-30.48" y1="154.94" x2="-38.1" y2="154.94" width="0.1524" layer="91"/>
+<wire x1="-38.1" y1="154.94" x2="-40.64" y2="154.94" width="0.1524" layer="91"/>
+<wire x1="-38.1" y1="149.86" x2="-38.1" y2="154.94" width="0.1524" layer="91"/>
+<pinref part="D1" gate="G$1" pin="C"/>
 </segment>
 </net>
@@
 <pinref part="R5" gate="G$1" pin="1"/>
 <pinref part="MASTER" gate="G$1" pin="DI"/>
-<pinref part="R8" gate="G$1" pin="2"/>
-<wire x1="-35.56" y1="119.38" x2="-25.4" y2="119.38" width="0.1524" layer="91"/>
-<wire x1="-48.26" y1="119.38" x2="-35.56" y2="119.38" width="0.1524" layer="91"/>
+<wire x1="-48.26" y1="119.38" x2="-25.4" y2="119.38" width="0.1524" layer="91"/>
 </segment>
 </net>
@@
 </segment>
 </net>
+<net name="N$5" class="0">
+<segment>
+<pinref part="MASTER" gate="G$1" pin="RO"/>
+<pinref part="R1" gate="G$1" pin="1"/>
+<wire x1="-25.4" y1="144.78" x2="-30.48" y2="144.78" width="0.1524" layer="91"/>
+</segment>
+</net>
