File: Schematic/Reciever_Reed.sch (EAGLE design)
At the start: 8 parts, among them IC1 ATMEGA328P, IC2 LTC485N, IC3 7805T, IC4 LM50

Commit message: Gør klar til eksamen
Parts:
- removed IC4: LM50, linear:LM50
- added R2: 10K, eagle-ltspice:R
- added S1: Reed Switch, switch-reed:REED-SWITCH-CT10-1530-G1
Connections:
- removed net N$1: IC1.PB5, IC2.!RE, IC2.DE
- removed net N$6: IC1.PC4, IC4.VO
- new net N$4: IC1.PD2, IC2.!RE, IC2.DE
- net GND: now also R2.2; no longer IC4.GND
- net N$3: now also S1.2
- net VCC: now also R2.1, S1.1; no longer IC4.+VS
Other:
- moved on the sheet: IC2, R1
Changed lines of the file:
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@@
 <part name="R1" library="eagle-ltspice" deviceset="R" device="" value="120"/>
 <part name="SUPPLY4" library="supply2" deviceset="GND" device=""/>
-<part name="IC4" library="linear" deviceset="LM50" device=""/>
 <part name="IC3" library="linear" deviceset="78*" device="T" technology="05"/>
 <part name="SUPPLY3" library="supply2" deviceset="GND" device=""/>
@@
 <part name="SUPPLY6" library="supply2" deviceset="VCC" device=""/>
 <part name="SUPPLY8" library="supply2" deviceset="VCC" device="" value="5V"/>
-<part name="SUPPLY7" library="supply2" deviceset="GND" device=""/>
 <part name="SUPPLY9" library="supply2" deviceset="VCC" device="" value="RX"/>
 <part name="SUPPLY10" library="supply2" deviceset="VCC" device="" value="RX"/>
 <part name="G1" library="battery" deviceset="BATTERY-HOLDER_11.6MM" device="" value=""/>
 <part name="SUPPLY11" library="supply2" deviceset="VCC" device="" value="5V"/>
+<part name="S1" library="switch-reed" deviceset="REED-SWITCH-" device="CT10-1530-G1" value="Reed Switch"/>
+<part name="SUPPLY7" library="supply2" deviceset="VCC" device="" value="5V"/>
+<part name="R2" library="eagle-ltspice" deviceset="R" device="" value="10K"/>
+<part name="SUPPLY12" library="supply2" deviceset="GND" device=""/>
 </parts>
 <sheets>
@@
 <instances>
 <instance part="IC1" gate="1" x="109.22" y="68.58"/>
-<instance part="IC2" gate="G$1" x="132.08" y="53.34"/>
+<instance part="IC2" gate="G$1" x="144.78" y="25.4"/>
 <instance part="SUPPLY1" gate="G$1" x="25.4" y="38.1" rot="R180"/>
 <instance part="SUPPLY2" gate="GND" x="66.04" y="55.88"/>
-<instance part="R1" gate="G$1" x="154.94" y="50.8" rot="R270"/>
-<instance part="SUPPLY4" gate="GND" x="142.24" y="45.72"/>
-<instance part="IC4" gate="G$1" x="149.86" y="73.66"/>
+<instance part="R1" gate="G$1" x="165.1" y="22.86" rot="R270"/>
+<instance part="SUPPLY4" gate="GND" x="154.94" y="15.24"/>
 <instance part="IC3" gate="A1" x="40.64" y="58.42"/>
 <instance part="SUPPLY3" gate="GND" x="40.64" y="38.1"/>
@@
 <instance part="SUPPLY5" gate="G$1" x="50.8" y="68.58"/>
 <instance part="SUPPLY6" gate="G$1" x="76.2" y="66.04" rot="R90"/>
-<instance part="SUPPLY8" gate="G$1" x="134.62" y="76.2"/>
-<instance part="SUPPLY7" gate="GND" x="149.86" y="63.5"/>
+<instance part="SUPPLY8" gate="G$1" x="154.94" y="35.56"/>
 <instance part="SUPPLY9" gate="G$1" x="73.66" y="101.6"/>
-<instance part="SUPPLY10" gate="G$1" x="121.92" y="58.42"/>
+<instance part="SUPPLY10" gate="G$1" x="134.62" y="33.02"/>
 <instance part="G1" gate="G$1" x="127" y="99.06"/>
 <instance part="SUPPLY11" gate="G$1" x="132.08" y="96.52" rot="R180"/>
+<instance part="S1" gate="G$1" x="119.38" y="45.72" rot="R270"/>
+<instance part="SUPPLY7" gate="G$1" x="127" y="53.34"/>
+<instance part="R2" gate="G$1" x="132.08" y="45.72"/>
+<instance part="SUPPLY12" gate="GND" x="137.16" y="43.18"/>
 </instances>
 <busses>
 </busses>
 <nets>
-<net name="N$1" class="0">
-<segment>
-<pinref part="IC1" gate="1" pin="PB5"/>
-<pinref part="IC2" gate="G$1" pin="DE"/>
-<wire x1="109.22" y1="50.8" x2="121.92" y2="50.8" width="0.1524" layer="91"/>
-<pinref part="IC2" gate="G$1" pin="!RE"/>
-<wire x1="121.92" y1="50.8" x2="121.92" y2="53.34" width="0.1524" layer="91"/>
-</segment>
-</net>
 <net name="GND" class="0">
 <segment>
@@
 <pinref part="IC2" gate="G$1" pin="GND"/>
 <pinref part="SUPPLY4" gate="GND" pin="GND"/>
+<wire x1="154.94" y1="20.32" x2="154.94" y2="17.78" width="0.1524" layer="91"/>
 </segment>
 <segment>
@@
 </segment>
 <segment>
-<pinref part="IC4" gate="G$1" pin="GND"/>
-<pinref part="SUPPLY7" gate="GND" pin="GND"/>
+<pinref part="R2" gate="G$1" pin="2"/>
+<pinref part="SUPPLY12" gate="GND" pin="GND"/>
 </segment>
 </net>
@@
 <segment>
 <pinref part="IC2" gate="G$1" pin="A"/>
-<wire x1="142.24" y1="53.34" x2="147.32" y2="53.34" width="0.1524" layer="91"/>
-<wire x1="147.32" y1="53.34" x2="147.32" y2="55.88" width="0.1524" layer="91"/>
+<wire x1="154.94" y1="25.4" x2="157.48" y2="25.4" width="0.1524" layer="91"/>
+<wire x1="157.48" y1="25.4" x2="160.02" y2="27.94" width="0.1524" layer="91"/>
 <pinref part="R1" gate="G$1" pin="1"/>
-<wire x1="147.32" y1="55.88" x2="154.94" y2="55.88" width="0.1524" layer="91"/>
-<wire x1="154.94" y1="55.88" x2="157.48" y2="55.88" width="0.1524" layer="91"/>
-<junction x="157.48" y="55.88"/>
-<label x="157.48" y="58.42" size="1.778" layer="95"/>
+<wire x1="160.02" y1="27.94" x2="165.1" y2="27.94" width="0.1524" layer="91"/>
+<wire x1="165.1" y1="27.94" x2="170.18" y2="27.94" width="0.1524" layer="91"/>
+<junction x="170.18" y="27.94"/>
+<label x="172.72" y="27.94" size="1.778" layer="95"/>
 </segment>
 </net>
@@
 <segment>
 <pinref part="IC2" gate="G$1" pin="B"/>
-<wire x1="142.24" y1="50.8" x2="147.32" y2="50.8" width="0.1524" layer="91"/>
 <pinref part="R1" gate="G$1" pin="2"/>
-<wire x1="154.94" y1="45.72" x2="147.32" y2="45.72" width="0.1524" layer="91"/>
-<wire x1="147.32" y1="45.72" x2="147.32" y2="50.8" width="0.1524" layer="91"/>
-<wire x1="154.94" y1="45.72" x2="157.48" y2="45.72" width="0.1524" layer="91"/>
-<junction x="157.48" y="45.72"/>
-<label x="157.48" y="43.18" size="1.778" layer="95"/>
+<wire x1="165.1" y1="17.78" x2="160.02" y2="22.86" width="0.1524" layer="91"/>
+<wire x1="160.02" y1="22.86" x2="154.94" y2="22.86" width="0.1524" layer="91"/>
+<wire x1="165.1" y1="17.78" x2="170.18" y2="17.78" width="0.1524" layer="91"/>
+<junction x="170.18" y="17.78"/>
+<label x="172.72" y="17.78" size="1.778" layer="95"/>
 </segment>
 </net>
@@
 <wire x1="55.88" y1="86.36" x2="78.74" y2="86.36" width="0.1524" layer="91"/>
 <pinref part="IC2" gate="G$1" pin="DI"/>
-<wire x1="121.92" y1="48.26" x2="121.92" y2="25.4" width="0.1524" layer="91"/>
-<wire x1="121.92" y1="25.4" x2="55.88" y2="25.4" width="0.1524" layer="91"/>
-<wire x1="55.88" y1="86.36" x2="55.88" y2="25.4" width="0.1524" layer="91"/>
+<wire x1="134.62" y1="20.32" x2="121.92" y2="22.86" width="0.1524" layer="91"/>
+<wire x1="121.92" y1="22.86" x2="55.88" y2="22.86" width="0.1524" layer="91"/>
+<wire x1="55.88" y1="86.36" x2="55.88" y2="22.86" width="0.1524" layer="91"/>
 </segment>
 </net>
@@
 <pinref part="IC1" gate="1" pin="PB4"/>
 <wire x1="109.22" y1="45.72" x2="114.3" y2="45.72" width="0.1524" layer="91"/>
+<pinref part="S1" gate="G$1" pin="2"/>
 </segment>
 </net>
@@
 </segment>
 <segment>
-<pinref part="IC4" gate="G$1" pin="+VS"/>
 <pinref part="SUPPLY8" gate="G$1" pin="VCC"/>
-<wire x1="134.62" y1="73.66" x2="139.7" y2="73.66" width="0.1524" layer="91"/>
 <pinref part="IC2" gate="G$1" pin="VCC"/>
-<wire x1="142.24" y1="55.88" x2="142.24" y2="66.04" width="0.1524" layer="91"/>
-<wire x1="142.24" y1="66.04" x2="134.62" y2="66.04" width="0.1524" layer="91"/>
-<wire x1="134.62" y1="66.04" x2="134.62" y2="73.66" width="0.1524" layer="91"/>
+<wire x1="154.94" y1="27.94" x2="154.94" y2="33.02" width="0.1524" layer="91"/>
 </segment>
 <segment>
@@
 <pinref part="IC2" gate="G$1" pin="RO"/>
 <pinref part="SUPPLY10" gate="G$1" pin="VCC"/>
+<wire x1="134.62" y1="27.94" x2="134.62" y2="30.48" width="0.1524" layer="91"/>
 </segment>
 <segment>
@@
 <pinref part="SUPPLY11" gate="G$1" pin="VCC"/>
 </segment>
-</net>
-<net name="N$6" class="0">
 <segment>
-<pinref part="IC4" gate="G$1" pin="VO"/>
-<wire x1="160.02" y1="73.66" x2="162.56" y2="73.66" width="0.1524" layer="91"/>
-<wire x1="162.56" y1="73.66" x2="162.56" y2="91.44" width="0.1524" layer="91"/>
-<pinref part="IC1" gate="1" pin="PC4"/>
-<wire x1="162.56" y1="91.44" x2="109.22" y2="91.44" width="0.1524" layer="91"/>
+<pinref part="S1" gate="G$1" pin="1"/>
+<wire x1="127" y1="45.72" x2="127" y2="50.8" width="0.1524" layer="91"/>
+<pinref part="SUPPLY7" gate="G$1" pin="VCC"/>
+<pinref part="R2" gate="G$1" pin="1"/>
+<junction x="127" y="45.72"/>
 </segment>
 </net>
@@
 </segment>
 </net>
+<net name="N$4" class="0">
+<segment>
+<pinref part="IC1" gate="1" pin="PD2"/>
+<wire x1="78.74" y1="81.28" x2="60.96" y2="81.28" width="0.1524" layer="91"/>
+<wire x1="60.96" y1="81.28" x2="60.96" y2="25.4" width="0.1524" layer="91"/>
+<pinref part="IC2" gate="G$1" pin="DE"/>
+<pinref part="IC2" gate="G$1" pin="!RE"/>
+<wire x1="119.38" y1="25.4" x2="134.62" y2="22.86" width="0.1524" layer="91"/>
+<wire x1="134.62" y1="22.86" x2="134.62" y2="25.4" width="0.1524" layer="91"/>
+<wire x1="60.96" y1="25.4" x2="119.38" y2="25.4" width="0.1524" layer="91"/>
+</segment>
+</net>
